File: Focus_Controller_Schematic.kicad_sch (KiCad schematic)
At the start: 3 parts, among them M1 Focus_Motor, U1 Stepper Motor Driver PK2

Commit message: complete controller schematic
Parts:
- removed A1: Arduino_UNO_R2, Module:Arduino_UNO_R2, symbol MCU_Module:Arduino_UNO_R2
- added A2: Arduino_UNO_R3, Module:Arduino_UNO_R3, symbol MCU_Module:Arduino_UNO_R3
- added Q1, Q2, Q3: BC547, Package_TO_SOT_THT:TO-92_Inline, symbol Transistor_BJT:BC547
- added R1, R2, R3: R, symbol Device:R
Connections:
- net at U1.7 (ENERGISE): now also Q3.1 (C)
- net at U1.8 (DIRECTION): now also Q2.1 (C)
- net at U1.9 (CLOCK_IN): now also Q1.1 (C)
- net GND: no longer names the net of U1.5 (0V)
- net GND: now also A2.29 (GND), Q1.3 (E), Q2.3 (E), Q3.3 (E)
- new net: Q3.2 (B), R1.1
- new net: A2.22 (D7), R1.2
- new net: Q2.2 (B), R2.1
- new net: A2.23 (D8), R2.2
- new net: A2.24 (D9), R3.2
- new net: Q1.2 (B), R3.1
- new net Lower Limit: A2.17 (D2)
- new net Upper Limit: A2.18 (D3)
Other:
- note added: "Legend:"
- moved on the sheet: M1
